File: Hardware/Photon_Proto_Shield.brd (EAGLE design)
At the start: 40.6 x 35.6 mm, 14 parts

Commit message: Changed per design review
Box around I2C breakout, moved sad and scale traces outside of photo
area, cleaned up silk on gnd and 3v3 busses.
Routing:
- net SCL: track 31.2 -> 36.2 mm
Changed lines of the file:
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@@
 <text x="4.318" y="0.381" size="1.016" layer="16" font="vector" ratio="15" rot="MR0">v10</text>
 <wire x1="15.494" y1="28.448" x2="17.018" y2="28.448" width="0.2032" layer="21"/>
-<wire x1="17.018" y1="28.448" x2="17.526" y2="28.956" width="0.2032" layer="21"/>
+<wire x1="17.018" y1="28.448" x2="17.653" y2="29.083" width="0.2032" layer="21"/>
 <wire x1="19.939" y1="28.448" x2="18.542" y2="28.448" width="0.2032" layer="21"/>
 <wire x1="18.542" y1="28.448" x2="17.907" y2="29.083" width="0.2032" layer="21"/>
-<wire x1="17.907" y1="29.083" x2="17.907" y2="29.21" width="0.2032" layer="21"/>
 <wire x1="23.241" y1="28.448" x2="24.765" y2="28.448" width="0.2032" layer="21"/>
-<wire x1="24.765" y1="28.448" x2="25.273" y2="28.956" width="0.2032" layer="21"/>
+<wire x1="24.765" y1="28.448" x2="25.4" y2="29.083" width="0.2032" layer="21"/>
 <wire x1="12.192" y1="28.448" x2="10.795" y2="28.448" width="0.2032" layer="21"/>
-<wire x1="10.795" y1="28.448" x2="10.16" y2="29.083" width="0.2032" layer="21"/>
-<wire x1="10.16" y1="29.083" x2="10.16" y2="29.21" width="0.2032" layer="21"/>
-<wire x1="12.192" y1="28.575" x2="10.668" y2="28.575" width="0.2032" layer="22"/>
-<wire x1="10.668" y1="28.575" x2="10.16" y2="29.21" width="0.2032" layer="22"/>
+<wire x1="10.795" y1="28.448" x2="10.16" y2="29.21" width="0.2032" layer="21"/>
+<wire x1="12.192" y1="28.448" x2="10.795" y2="28.448" width="0.2032" layer="22"/>
+<wire x1="10.795" y1="28.448" x2="10.16" y2="29.21" width="0.2032" layer="22"/>
 <wire x1="15.494" y1="28.448" x2="17.018" y2="28.448" width="0.2032" layer="22"/>
-<wire x1="17.018" y1="28.448" x2="17.526" y2="28.956" width="0.2032" layer="22"/>
-<wire x1="19.939" y1="28.448" x2="18.415" y2="28.448" width="0.2032" layer="22"/>
-<wire x1="18.415" y1="28.448" x2="17.78" y2="29.083" width="0.2032" layer="22"/>
+<wire x1="17.018" y1="28.448" x2="17.653" y2="29.083" width="0.2032" layer="22"/>
+<wire x1="19.939" y1="28.448" x2="18.542" y2="28.448" width="0.2032" layer="22"/>
+<wire x1="18.542" y1="28.448" x2="17.907" y2="29.083" width="0.2032" layer="22"/>
 <wire x1="23.241" y1="28.448" x2="24.765" y2="28.448" width="0.2032" layer="22"/>
-<wire x1="24.765" y1="28.448" x2="25.273" y2="28.956" width="0.2032" layer="22"/>
+<wire x1="24.765" y1="28.448" x2="25.4" y2="29.083" width="0.2032" layer="22"/>
 <text x="12.192" y="33.909" size="1.016" layer="22" font="vector" ratio="15" rot="MR0">I2C</text>
 <text x="19.05" y="-12.7" size="1.778" layer="51" font="vector" ratio="10">Ben Leduc-Mills</text>
 <text x="36.83" y="17.78" size="1.27" layer="22" font="vector" ratio="15" rot="MR270" align="bottom-center">Proto Shield
 for the Photon</text>
+<wire x1="9.652" y1="35.56" x2="9.652" y2="33.528" width="0.2032" layer="21"/>
+<wire x1="9.652" y1="33.528" x2="11.43" y2="31.75" width="0.2032" layer="21"/>
+<wire x1="11.43" y1="31.75" x2="23.622" y2="31.75" width="0.2032" layer="21"/>
+<wire x1="23.622" y1="31.75" x2="23.622" y2="35.56" width="0.2032" layer="21"/>
+<wire x1="23.622" y1="35.56" x2="23.495" y2="35.56" width="0.2032" layer="21"/>
 </plain>
 <attributes>
@@
 <contactref element="JP1" pad="D1"/>
 <contactref element="JP2" pad="4"/>
-<wire x1="26.67" y1="6.35" x2="25.4" y2="7.62" width="0.2032" layer="16"/>
-<wire x1="25.4" y1="7.62" x2="23.368" y2="7.62" width="0.2032" layer="16"/>
-<wire x1="23.368" y1="7.62" x2="22.86" y2="8.128" width="0.2032" layer="16"/>
-<wire x1="22.86" y1="8.128" x2="22.86" y2="33.02" width="0.2032" layer="16"/>
+<wire x1="29.21" y1="7.62" x2="29.21" y2="32.258" width="0.2032" layer="16"/>
 <wire x1="22.86" y1="33.02" x2="21.59" y2="34.29" width="0.2032" layer="16"/>
+<wire x1="26.67" y1="6.35" x2="27.94" y2="6.35" width="0.2032" layer="16"/>
+<wire x1="27.94" y1="6.35" x2="29.21" y2="7.62" width="0.2032" layer="16"/>
+<wire x1="29.21" y1="32.258" x2="28.448" y2="33.02" width="0.2032" layer="16"/>
+<wire x1="28.448" y1="33.02" x2="22.86" y2="33.02" width="0.2032" layer="16"/>
 </signal>
 <signal name="SDA">
@@
 <contactref element="JP2" pad="3"/>
 <wire x1="26.67" y1="3.81" x2="25.4" y2="5.08" width="0.2032" layer="16"/>
-<wire x1="19.05" y1="34.29" x2="20.32" y2="33.02" width="0.2032" layer="16"/>
-<wire x1="20.32" y1="33.02" x2="20.32" y2="5.715" width="0.2032" layer="16"/>
-<wire x1="20.32" y1="5.715" x2="20.955" y2="5.08" width="0.2032" layer="16"/>
-<wire x1="20.955" y1="5.08" x2="25.4" y2="5.08" width="0.2032" layer="16"/>
+<wire x1="19.05" y1="34.29" x2="20.955" y2="32.385" width="0.2032" layer="16"/>
+<wire x1="25.4" y1="31.75" x2="25.4" y2="5.08" width="0.2032" layer="16"/>
+<wire x1="25.4" y1="31.75" x2="24.765" y2="32.385" width="0.2032" layer="16"/>
+<wire x1="24.765" y1="32.385" x2="20.955" y2="32.385" width="0.2032" layer="16"/>
 </signal>
 <signal name="VCC">
